File: Pikatea Top Pro Micro/PikateaTPM.sch (KiCad schematic (older format))
At the start: 22 parts, among them J1 USB_B_Mini, J2 Conn_01x08, J3 Conn_01x08, J4 Conn_01x05, J6 AVR-ISP-6, J7 01x15, U1 ATmega32U4, X1 16MHz

Commit message: Remove R6 and rename MCU data line nets
Parts:
- removed R6: 10k, Resistor_SMD:R_0402_1005Metric, symbol Device:R
Connections:
- net MCU_D+: now reaches R4.1, U1.4 (D+)
- net MCU_D-: now reaches R5.1, U1.3 (D-)
Changed lines of the file:
@@
 EESchema Schematic File Version 4
-EELAYER 30 0
+LIBS:PikateaTPM-cache
+EELAYER 26 0
 EELAYER END
 $Descr A4 11693 8268
@@
 Wire Wire Line
 	6300 1400 6600 1400
-$Comp
-L Device:R R6
-U 1 1 5CBBA935
-P 6900 1150
-F 0 "R6" V 6980 1150 50  0000 C CNN
-F 1 "10k" V 6900 1150 50  0000 C CNN
-F 2 "Resistor_SMD:R_0402_1005Metric" V 6830 1150 50  0001 C CNN
-F 3 "" H 6900 1150 50  0001 C CNN
-F 4 "C25744" V 6900 1150 50  0001 C CNN "LCSC"
-	1    6900 1150
-	-1   0    0    1
-$EndComp
-Wire Wire Line
-	6900 1000 6900 900
-Wire Wire Line
-	6900 900  6600 900
-Connection ~ 6600 900
-Wire Wire Line
-	6900 1300 6900 1400
-Wire Wire Line
-	6900 1400 6600 1400
-Connection ~ 6600 1400
 Text Label 10350 3500 0    60   ~ 0
 PD5
@@
 Wire Wire Line
 	4100 3100 4350 3100
+Text Label 7500 3150 2    60   ~ 0
+MCU_D+
+Text Label 7600 3250 2    60   ~ 0
+MCU_D-
 $EndSCHEMATC

Commit message: Change MCU footprint to QFP-44_10x10x08P
Parts:
- U1: footprint Package_DFN_QFN:QFN-44-1EP_7x7mm_P0.5mm_EP5.2x5.2mm -> Package_QFP:TQFP-44_10x10mm_P0.8mm
Changed lines of the file:
@@
 F 0 "U1" H 8200 5050 50  0000 C CNN
 F 1 "ATmega32U4" H 9850 1850 50  0000 C CNN
-F 2 "Package_DFN_QFN:QFN-44-1EP_7x7mm_P0.5mm_EP5.2x5.2mm" H 9150 3350 50  0001 C CIN
+F 2 "Package_QFP:TQFP-44_10x10mm_P0.8mm" H 9150 3350 50  0001 C CIN
 F 3 "" H 10250 4450 50  0001 C CNN
 F 4 "C44854" H 9150 3350 50  0001 C CNN "LCSC"
