File: Pikatea Macropad Mini/Pikatea Macropad Mini.kicad_pcb (KiCad board)
At the start: 2 copper layers, 126.1 x 25 mm, 39 parts, among them J1 AVR-ISP-6, J2 Conn_01x02_Male, J3 Conn_01x02_Male, J4 Conn_01x03_Male, J5 Conn_01x03_Male, SW1 SW_DPST, SW2 Rotary_Encoder_Switch, SW3 SW_SPST, U1 ATMEGA32U4-EP, U2 AMS1117-3.3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

Commit message: updated gerbers
Other:
- board size 126.1 x 25 mm -> 125.1 x 25 mm

Commit message: added more projects
Parts:
- added J6: Conn_01x04_Male, Pikatea Macropad Encoder Side Mount:Breakaway-Throughole, F.Cu at (177.5, 106.0)
- moved J4 2.56 mm to (174.6, 91.5)
Routing:
- net GND: track 190.6 -> 205.6 mm
- net /D1: track 32.7 -> 30.0 mm
- net /D0: track 33.4 -> 31.0 mm
- net /A0: track 140.0 -> 141.4 mm
Other:
- outline, holes or cut-outs redrawn
