File: Pikatea Macropad Mini/Pikatea Macropad Mini.sch (KiCad schematic (older format))
At the start: 31 parts, among them SW1 SW_DPST, SW2 Rotary_Encoder_Switch, U1 ATMEGA32U4-EP, U2 AMS1117-3.3, U3 74LVC125APW,118, X1 16MHz

Commit message: completed mini version 1
Parts:
- added J1: AVR-ISP-6, Connector_IDC:IDC-Header_2x03_P2.54mm_Vertical, symbol Connector:AVR-ISP-6
- added J2, J3: Conn_01x02_Male, Connector_PinHeader_2.54mm:PinHeader_1x02_P2.54mm_Vertical, symbol Connector:Conn_01x02_Male
- added J4, J5: Conn_01x03_Male, Connector_PinHeader_2.54mm:PinHeader_1x03_P2.54mm_Vertical, symbol Connector:Conn_01x03_Male
- added MX4, MX5: MX-NoLED, Button_Switch_Keyboard:SW_Cherry_MX_1.00u_PCB, symbol MX_Alps_Hybrid:MX-NoLED
- added SW3: SW_SPST, Pikatea Macropad Encoder Side Mount:Pikatea_Solder_switch, symbol Switch:SW_SPST
- C1, C10, C11, C12, C13, C14, C2, C3, C4, C5, C6, C7, C8, C9: footprint (none) -> Capacitor_SMD:C_0805_2012Metric
- MX1, MX2, MX3: footprint (none) -> Button_Switch_Keyboard:SW_Cherry_MX_1.00u_PCB
- R1, R2, R3, R4, R5, R6, R7: footprint (none) -> Resistor_SMD:R_0805_2012Metric
- SW1: footprint (none) -> Button_Switch_SMD:SW_SPST_TL3342
- SW2: footprint (none) -> Pikatea Macropad Encoder Side Mount:Encoder-BI_EN11_HSM0E
- U1: footprint QFN44 -> Package_QFP:LQFP-44_10x10mm_P0.8mm
- U3: footprint SOP65P640X110-14N -> Package_SO:TSSOP-14-1EP_4.4x5mm_P0.65mm
- X1: footprint (none) -> Crystal:Crystal_SMD_SeikoEpson_FA238-4Pin_3.2x2.5mm
- XS1: footprint Connectors:Conn_uSDcard -> Pikatea_SDcard_reader:XUNPU_TF-110
Connections:
- net labels added: D0, D1, D11, D12, D13
- wire segments 119 -> 145
- no-connect marks 2 -> 6
Other:
- moved on the sheet: SW1

Commit message: added more projects
Parts:
- added J6: Conn_01x04_Male, Pikatea Macropad Encoder Side Mount:Breakaway-Throughole, symbol Connector:Conn_01x04_Male
Connections:
- wire segments 145 -> 146
Changed lines of the file:
@@
 Text Label 6900 2000 0    50   ~ 0
 D6
+Text Label 5750 1900 0    50   ~ 0
+D8
+Text Label 5750 2000 0    50   ~ 0
+D6
+Wire Wire Line
+	5750 2100 6500 2100
+Connection ~ 6500 2100
+$Comp
+L Connector:Conn_01x04_Male J6
+U 1 1 601C442B
+P 5550 1900
+F 0 "J6" H 5658 2181 50  0000 C CNN
+F 1 "Conn_01x04_Male" H 5658 2090 50  0000 C CNN
+F 2 "Pikatea Macropad Encoder Side Mount:Breakaway-Throughole" H 5550 1900 50  0001 C CNN
+F 3 "~" H 5550 1900 50  0001 C CNN
+	1    5550 1900
+	1    0    0    -1
+$EndComp
+$Comp
+L power:GND #PWR?
+U 1 1 601CF47F
+P 5750 1800
+F 0 "#PWR?" H 5750 1550 50  0001 C CNN
+F 1 "GND" V 5755 1672 50  0000 R CNN
+F 2 "" H 5750 1800 50  0001 C CNN
+F 3 "" H 5750 1800 50  0001 C CNN
+	1    5750 1800
+	0    -1   -1   0
+$EndComp
 $EndSCHEMATC
