File: Pikatea SD card Module/Pikatea SD card Module.kicad_pcb (KiCad board)
At the start: 2 copper layers, 37 x 14.5 mm, 13 parts, among them J1 Conn_01x03_Male, J2 Conn_01x03_Male, U1 AMS1117-3.3, U2 74LVC125APW,118

Commit message: changes
Parts:
- C3: value 100uF -> 10uF
- moved C1 0.40 mm to (213.9, 75.1), turned to 30 degrees
Connections:
- J2 pad 2: Net-(J2-Pad2) -> MISO
Routing:
- net MISO: track 0.00 -> 7.67 mm, vias 0 -> 2
- net Net-(J2-Pad2): track 0.86 -> 0.00 mm
- net GND: track 55.4 -> 56.1 mm
Other:
- board text added: "Pikatea SDcM-2"
- board text removed: "Pikatea SDcM-1"
