File: Pikatea SD card Module/Pikatea SD card Module.sch (KiCad schematic (older format))
At the start: 13 parts, among them J1 Conn_01x03_Male, J2 Conn_01x03_Male, U1 AMS1117-3.3, U2 74LVC125APW,118

Commit message: changes
Changed lines of the file:
@@
 Text GLabel 7800 3450 2    50   Input ~ 0
 SCK
+Text GLabel 7800 4150 2    50   Input ~ 0
+MISO
 $EndSCHEMATC
