File: Pikatea Macropad GB3/Pikatea Macropad GB3.kicad_pcb (KiCad board)
At the start: 2 copper layers, 125.1 x 25.2 mm, 27 parts, among them J1 TC2030-CTX, J2 USB_B_Mini, J4 Conn_01x03_Male, J5 Conn_01x03_Male, J6 Conn_01x04_Male, SW1 SW_DPST, SW2 Rotary_Encoder_Switch, U1 ATMEGA32U4-EP, X1 16MHz

Commit message: changes
Parts:
- added J3: Conn_01x03_Male, Connector_PinHeader_2.54mm:PinHeader_1x03_P2.54mm_Vertical, F.Cu at (140.0, 107.2)
- added J7: Conn_01x03_Male, Connector_PinHeader_2.54mm:PinHeader_1x03_P2.54mm_Vertical, F.Cu at (160.0, 107.2)
- moved C7 84.6 mm to (108.6, 97.0), turned to 180 degrees
- moved C3 81.7 mm to (112.2, 104.9), turned to 180 degrees
- moved C5 73.9 mm to (122.8, 105.2)
- moved C8 70.7 mm to (108.4, 90.7)
- moved C10 69.2 mm to (124.6, 102.6)
- moved J4 68.3 mm to (114.0, 107.4), turned to 0 degrees
- moved C1 67.8 mm to (112.6, 89.9), turned to 180 degrees
- moved R3 66.5 mm to (111.5, 111.7), turned to 270 degrees
- moved C4 61.4 mm to (126.7, 100.6)
- moved C6 60.4 mm to (127.2, 96.0), turned to 270 degrees
- moved C2 59.8 mm to (123.3, 89.9)
- moved C9 58.7 mm to (127.6, 89.9)
- moved R4 53.7 mm to (130.0, 92.2), turned to 180 degrees
- moved R5 47.5 mm to (130.0, 94.7), turned to 180 degrees
- moved X1 17.0 mm to (108.4, 93.9)
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Routing:
- net GND: track 0.00 -> 147.5 mm, vias 0 -> 12
- net VBUS: track 0.00 -> 135.1 mm, vias 0 -> 9
- net /A0: track 0.06 -> 124.4 mm, vias 0 -> 2
- net /D6: track 0.00 -> 104.1 mm, vias 0 -> 2
- net /D8: track 0.00 -> 95.9 mm, vias 0 -> 1
- net /RESET: track 0.00 -> 89.7 mm, vias 0 -> 3
- net /MISO: track 0.00 -> 75.2 mm, vias 0 -> 5
- net /SCK: track 0.00 -> 59.8 mm, vias 0 -> 2
- net /D7: track 0.00 -> 53.2 mm, vias 0 -> 2
- net /MOSI: track 0.00 -> 51.0 mm, vias 0 -> 3
- net /D3: track 0.00 -> 49.6 mm, vias 0 -> 1
- net /D9: track 0.00 -> 44.1 mm, vias 0 -> 1
- net /D4: track 0.00 -> 35.1 mm, vias 0 -> 1
- net /CS: track 0.00 -> 32.5 mm, vias 0 -> 2
- net /D1: track 0.00 -> 16.9 mm, vias 0 -> 1
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Other:
- outline, holes or cut-outs redrawn
- board text added: "A"
- board text added: "Pikatea Macropad GB3"

Commit message: updates
Parts:
- J1: value TC2030-CTX -> AVR-ISP-6; footprint TC2030-CTX:TC2030-IDC -> keyboard_parts:AVR_ICSP_3x2
- moved J1 0.91 mm to (100.3, 95.0)
- moved J3 0.50 mm to (140.0, 106.7)
- moved J7 0.50 mm to (160.0, 106.7)
Connections:
- J1 pad 1: VBUS -> /MISO
- J1 pad 2: /MOSI -> VBUS
- J1 pad 3: /RESET -> /SCK
- J1 pad 4: /SCK -> /MOSI
- J1 pad 5: GND -> /RESET
- J1 pad 6: /MISO -> GND
- U1 pad 20: /D0 -> Net-(U1-Pad20)
- U1 pad 21: /D1 -> Net-(U1-Pad21)
- U1 pad 40: Net-(U1-Pad40) -> /D1
- U1 pad 41: Net-(U1-Pad41) -> /D0
Routing:
- net /D0: track 13.8 -> 21.9 mm, vias 1 -> 3
- net VBUS: track 135.1 -> 127.1 mm, vias 9 -> 8
- net /D1: track 16.9 -> 22.9 mm, vias 1 -> 3
- net /RESET: track 89.7 -> 83.8 mm
- net /D6: track 104.1 -> 98.4 mm
- net /MISO: track 75.2 -> 70.7 mm
- net /MOSI: track 51.0 -> 52.1 mm, vias 3 -> 2
- net /D7: track 53.2 -> 54.1 mm
- net GND: track 147.5 -> 148.2 mm, vias 12 -> 11
- net /CS: track 32.5 -> 33.1 mm
- net Net-(U1-Pad21): track 0.00 -> 0.59 mm
- net /SCK: track 59.8 -> 60.0 mm, vias 2 -> 1

Commit message: update gb3
Parts:
- J6: value Conn_01x04_Male -> Conn_01x06_Male
- moved J4 98.6 mm to (212.6, 107.3)
Connections:
- J4 pad 1: /D0 -> /D1
- J4 pad 2: /D1 -> /D0
Routing:
- net /D0: track 21.9 -> 120.6 mm, vias 3 -> 1
- net /D1: track 22.9 -> 119.3 mm, vias 3 -> 1
- net GND: track 148.2 -> 155.5 mm, vias 11 -> 13
- net /A0: track 124.4 -> 128.5 mm
- net /D8: track 95.9 -> 95.0 mm
