File: Pikatea Macropad GB3/Pikatea Macropad GB3.sch (KiCad schematic (older format))
At the start: 27 parts, among them J1 TC2030-CTX, J2 USB_B_Mini, J4 Conn_01x03_Male, J5 Conn_01x03_Male, J6 Conn_01x04_Male, SW1 SW_DPST, SW2 Rotary_Encoder_Switch, U1 ATMEGA32U4-EP, X1 16MHz

Commit message: changes
Parts:
- added J3, J7: Conn_01x03_Male, Connector_PinHeader_2.54mm:PinHeader_1x03_P2.54mm_Vertical, symbol Connector:Conn_01x03_Male
Connections:
- net CS: now also J3.3 (Pin_3)
- net GND: now also J7.1 (Pin_1)
- net MISO: now also J7.2 (Pin_2)
- net MOSI: now also J3.2 (Pin_2)
- net SCK: now also J3.1 (Pin_1)
- net VBUS: now also J7.3 (Pin_3)
Changed lines of the file:
@@
 	1    0    0    -1
 $EndComp
+$Comp
+L Connector:Conn_01x03_Male J3
+U 1 1 60614122
+P 3050 1750
+F 0 "J3" H 3158 2031 50  0000 C CNN
+F 1 "Conn_01x03_Male" H 3158 1940 50  0000 C CNN
+F 2 "Connector_PinHeader_2.54mm:PinHeader_1x03_P2.54mm_Vertical" H 3050 1750 50  0001 C CNN
+F 3 "~" H 3050 1750 50  0001 C CNN
+	1    3050 1750
+	1    0    0    -1
+$EndComp
+$Comp
+L Connector:Conn_01x03_Male J7
+U 1 1 606149C4
+P 3950 1750
+F 0 "J7" H 4058 2031 50  0000 C CNN
+F 1 "Conn_01x03_Male" H 4058 1940 50  0000 C CNN
+F 2 "Connector_PinHeader_2.54mm:PinHeader_1x03_P2.54mm_Vertical" H 3950 1750 50  0001 C CNN
+F 3 "~" H 3950 1750 50  0001 C CNN
+	1    3950 1750
+	1    0    0    -1
+$EndComp
+Text Label 3250 1650 0    50   ~ 0
+SCK
+Text Label 3250 1750 0    50   ~ 0
+MOSI
+Text Label 3250 1850 0    50   ~ 0
+CS
+Text Label 4150 1750 0    50   ~ 0
+MISO
+$Comp
+L power:GND #PWR0102
+U 1 1 6061DB34
+P 4150 1650
+F 0 "#PWR0102" H 4150 1400 50  0001 C CNN
+F 1 "GND" H 4155 1477 50  0000 C CNN
+F 2 "" H 4150 1650 50  0001 C CNN
+F 3 "" H 4150 1650 50  0001 C CNN
+	1    4150 1650
+	-1   0    0    1
+$EndComp
+$Comp
+L power:VCC #PWR0114
+U 1 1 606210F2
+P 4150 1850
+F 0 "#PWR0114" H 4150 1700 50  0001 C CNN
+F 1 "VCC" V 4165 1978 50  0000 L CNN
+F 2 "" H 4150 1850 50  0001 C CNN
+F 3 "" H 4150 1850 50  0001 C CNN
+	1    4150 1850
+	0    1    1    0
+$EndComp
 $EndSCHEMATC

Commit message: updates
Parts:
- removed J1: TC2030-CTX, TC2030-CTX:TC2030-IDC, symbol TC2030-CTX:TC2030-CTX
- added J1: AVR-ISP-6, keyboard_parts:AVR_ICSP_3x2, symbol Connector:AVR-ISP-6
Connections:
- net D0: now also U1.41 ((ADC0)PF0); no longer U1.20 ((RXD/INT2)PD2)
- net D1: now also U1.40 ((ADC1)PF1); no longer U1.21 ((TXD/INT3)PD3)
- net GND: now also J1.6 (GND)
- net MISO: now also J1.1 (MISO)
- net MOSI: now also J1.4 (MOSI)
- net RESET: now also J1.5 (~RST)
- net SCK: now also J1.3 (SCK)
- net VBUS: now also J1.2 (VCC)
Changed lines of the file:
@@
 	1    0    0    -1
 $EndComp
-Text Label 10850 3100 0    50   ~ 0
+Text Label 10700 2000 0    50   ~ 0
 MISO
-Text Label 10850 2900 0    50   ~ 0
+Text Label 10700 2100 0    50   ~ 0
 MOSI
-Text Label 10850 3000 0    50   ~ 0
+Text Label 10700 2200 0    50   ~ 0
 SCK
-Text Label 10850 3200 0    50   ~ 0
+Text Label 10700 2300 0    50   ~ 0
 RESET
 $Comp
 L power:GND #PWR0117
 U 1 1 600979DD
-P 9850 3200
-F 0 "#PWR0117" H 9850 2950 50  0001 C CNN
-F 1 "GND" H 9855 3027 50  0000 C CNN
-F 2 "" H 9850 3200 50  0001 C CNN
-F 3 "" H 9850 3200 50  0001 C CNN
-	1    9850 3200
+P 10200 2600
+F 0 "#PWR0117" H 10200 2350 50  0001 C CNN
+F 1 "GND" H 10205 2427 50  0000 C CNN
+F 2 "" H 10200 2600 50  0001 C CNN
+F 3 "" H 10200 2600 50  0001 C CNN
+	1    10200 2600
 	0    1    1    0
 $EndComp
@@
 L power:VCC #PWR0118
 U 1 1 60098DB5
-P 9850 2900
-F 0 "#PWR0118" H 9850 2750 50  0001 C CNN
-F 1 "VCC" V 9867 3028 50  0000 L CNN
-F 2 "" H 9850 2900 50  0001 C CNN
-F 3 "" H 9850 2900 50  0001 C CNN
-	1    9850 2900
+P 10200 1700
+F 0 "#PWR0118" H 10200 1550 50  0001 C CNN
+F 1 "VCC" V 10217 1828 50  0000 L CNN
+F 2 "" H 10200 1700 50  0001 C CNN
+F 3 "" H 10200 1700 50  0001 C CNN
+	1    10200 1700
 	0    -1   -1   0
 $EndComp
@@
 Text Label 8200 4050 0    50   ~ 0
 D13
-Text Label 8200 4450 0    50   ~ 0
+Text Label 8200 5450 0    50   ~ 0
 D0
-Text Label 8200 4550 0    50   ~ 0
+Text Label 8200 5550 0    50   ~ 0
 D1
 Text Label 8200 4850 0    50   ~ 0
@@
 Connection ~ 8650 1950
 $Comp
-L TC2030-CTX:TC2030-CTX J1
-U 1 1 60609235
-P 10350 3000
-F 0 "J1" H 10350 3367 50  0000 C CNN
-F 1 "TC2030-CTX" H 10350 3276 50  0000 C CNN
-F 2 "TC2030-CTX:TC2030-IDC" H 10350 3000 50  0001 C CNN
-F 3 "" H 10350 3000 50  0001 L BNN
-	1    10350 3000
-	1    0    0    -1
-$EndComp
-$Comp
 L Connector:Conn_01x03_Male J3
 U 1 1 60614122
@@
 	0    1    1    0
 $EndComp
+$Comp
+L Connector:AVR-ISP-6 J1
+U 1 1 6089E8EE
+P 10300 2200
+F 0 "J1" H 9971 2296 50  0000 R CNN
+F 1 "AVR-ISP-6" H 9971 2205 50  0000 R CNN
+F 2 "keyboard_parts:AVR_ICSP_3x2" V 10050 2250 50  0001 C CNN
+F 3 " ~" H 9025 1650 50  0001 C CNN
+	1    10300 2200
+	1    0    0    -1
+$EndComp
 $EndSCHEMATC

Commit message: update gb3
Parts:
- removed J6: Conn_01x04_Male, Pikatea Macropad Encoder Side Mount:Breakaway-Throughole, symbol Connector:Conn_01x04_Male
- added J6: Conn_01x06_Male, Pikatea Macropad Encoder Side Mount:Breakaway-Throughole, symbol Connector:Conn_01x06_Male
Connections:
- net A0: now also J6.4 (Pin_4)
- net D0: now also J4.2 (Pin_2), J6.6 (Pin_6); no longer J4.1 (Pin_1)
- net D1: now also J4.1 (Pin_1), J6.5 (Pin_5); no longer J4.2 (Pin_2)
- net D6: now also J6.3 (Pin_3)
- net D8: now also J6.2 (Pin_2)
- net GND: now also J6.1 (Pin_1)
Changed lines of the file:
@@
 Wire Wire Line
 	6500 2100 6900 2100
+Text Label 6500 2000 0    50   ~ 0
+D0
 Text Label 6500 1900 0    50   ~ 0
-D0
-Text Label 6500 2000 0    50   ~ 0
 D1
 Text Label 8200 3750 0    50   ~ 0
@@
 Connection ~ 6500 2100
 $Comp
-L Connector:Conn_01x04_Male J6
-U 1 1 601C442B
-P 5550 1900
-F 0 "J6" H 5658 2181 50  0000 C CNN
-F 1 "Conn_01x04_Male" H 5658 2090 50  0000 C CNN
-F 2 "Pikatea Macropad Encoder Side Mount:Breakaway-Throughole" H 5550 1900 50  0001 C CNN
-F 3 "~" H 5550 1900 50  0001 C CNN
-	1    5550 1900
-	1    0    0    -1
-$EndComp
-$Comp
 L power:GND #PWR0101
 U 1 1 601CF47F
@@
 	1    0    0    -1
 $EndComp
+$Comp
+L Connector:Conn_01x06_Male J6
+U 1 1 60A0116B
+P 5550 2000
+F 0 "J6" H 5658 2381 50  0000 C CNN
+F 1 "Conn_01x06_Male" H 5658 2290 50  0000 C CNN
+F 2 "Pikatea Macropad Encoder Side Mount:Breakaway-Throughole" H 5550 2000 50  0001 C CNN
+F 3 "~" H 5550 2000 50  0001 C CNN
+	1    5550 2000
+	1    0    0    -1
+$EndComp
+Text Label 5750 2300 0    50   ~ 0
+D0
+Text Label 5750 2200 0    50   ~ 0
+D1
 $EndSCHEMATC

Commit message: start finngus project
Changed lines of the file:
@@
 L power:GND #PWR0106
 U 1 1 5FC36DC8
-P 5400 3800
-F 0 "#PWR0106" H 5400 3550 50  0001 C CNN
-F 1 "GND" H 5405 3627 50  0000 C CNN
-F 2 "" H 5400 3800 50  0001 C CNN
-F 3 "" H 5400 3800 50  0001 C CNN
-	1    5400 3800
+P 5400 3900
+F 0 "#PWR0106" H 5400 3650 50  0001 C CNN
+F 1 "GND" H 5405 3727 50  0000 C CNN
+F 2 "" H 5400 3900 50  0001 C CNN
+F 3 "" H 5400 3900 50  0001 C CNN
+	1    5400 3900
 	1    0    0    -1
 $EndComp
@@
 Text Label 5750 2200 0    50   ~ 0
 D1
+Wire Wire Line
+	5400 3800 5400 3900
 $EndSCHEMATC
