File: Pikatea Keyboard/Pikatea Keyboard - Copy.kicad_pcb (KiCad board)
At the start: 2 copper layers, 319.6 x 93.7 mm, 170 parts, among them J1 AVR-ISP-6, J2 USB_B_Mini, SW1 SW_DPST, SW2 Rotary_Encoder_Switch, U1 ATMEGA32U4-EP, X1 16MHz

Commit message: update keyboard
Parts:
- removed D70: D_Small, Diode_SMD:D_SOD-123
- removed MX_LALT2, MX_LCTRL2, MX_RCTRL2: MX-LED, MX_Only:MXOnly-1.5U-FLIPPED
- removed MX_LEFT3, MX_UP2: MX-LED, MX_Only:MXOnly-1U
- removed MX_LMENU2, MX_RCTRL3, MX_RMENU2, MX_RMENU3: MX-LED, MX_Only:MXOnly-1U-FLIPPED
- removed MX_RSHFT2: MX-LED, MX_Only:MXOnly-1.75U-FLIPPED
- removed MX_SPACE2: MX-LED, MX_Only:MXOnly-7U-FLIPPED-ReversedStabilizers
- MX_LEFT1: footprint MX_Only:MXOnly-1.25U-FLIPPED -> MX_Only:MXOnly-1U
- MX_LEFT2: footprint MX_Only:MXOnly-1.5U-FLIPPED -> MX_Only:MXOnly-1.25U-FLIPPED
- moved D47 15.9 mm to (2.65, 87.2), turned to 270 degrees
- moved D30 7.23 mm to (102.7, 85.9), turned to 270 degrees
- moved D11 7.19 mm to (216.1, 85.8), turned to 270 degrees
- moved D27 7.14 mm to (122.1, 85.9), turned to 270 degrees
- moved D14 7.09 mm to (198.3, 85.8), turned to 270 degrees
- moved D33 6.96 mm to (84.4, 86.2), turned to 270 degrees
- moved D20 6.86 mm to (160.5, 86.2), turned to 270 degrees
- moved D7 6.84 mm to (236.7, 86.0), turned to 270 degrees
- moved D17 6.78 mm to (179.1, 85.9), turned to 270 degrees
- moved D2 6.62 mm to (259.1, 86.0), turned to 270 degrees
- moved D37 6.57 mm to (65.5, 86.4), turned to 270 degrees
- moved D23 6.37 mm to (140.4, 86.4), turned to 270 degrees
- moved D41 3.61 mm to (46.2, 86.1), turned to 270 degrees
- moved D44 3.36 mm to (27.4, 87.2), turned to 270 degrees
Connections:
- U1 pad 25: Col3 -> Net-(U1-Pad25)
- U1 pad 26: Col4 -> Net-(U1-Pad26)
- U1 pad 27: Col5 -> Net-(U1-Pad27)
Routing:
- net Col5: track 151.8 -> 87.4 mm
- net Col4: track 125.2 -> 81.1 mm
- net Col3: track 113.9 -> 94.9 mm
- net Net-(D47-Pad2): track 14.1 -> 4.79 mm, vias 1 -> 0
- net Net-(D37-Pad2): track 7.09 -> 3.53 mm
- net Net-(D33-Pad2): track 6.87 -> 3.61 mm
- net Net-(D20-Pad2): track 6.73 -> 3.68 mm
- net Net-(D7-Pad2): track 6.55 -> 3.76 mm
- net Net-(D14-Pad2): track 6.87 -> 4.09 mm
- net Net-(D27-Pad2): track 6.76 -> 4.03 mm
- net Net-(D17-Pad2): track 6.87 -> 4.16 mm
- net Net-(D30-Pad2): track 7.10 -> 4.42 mm
- net Net-(D23-Pad2): track 6.95 -> 4.80 mm
- net Row2: track 256.3 -> 257.9 mm
- net Net-(D44-Pad2): track 5.36 -> 3.84 mm
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