File: Pikatea Keyboard/Pikatea Keyboard.sch (KiCad schematic (older format))
At the start: 87 parts, among them J1 AVR-ISP-6, J2 USB_B_Mini, SW1 SW_DPST, SW2 Rotary_Encoder_Switch, U1 ATMEGA32U4-EP, X1 16MHz

Commit message: update keyboard
Parts:
- added D1, D10, D11, D12, D13, D14, D15, D16, D17, D18, D19, D2, D20, D21, D22, D23, D24, D25, D26, D27, D28, D29, D3, D30, D31, D32, D33, D34, D35, D36, D37, D38, D39, D4, D40, D41, D42, D43, D44, D45, D46, D47, D48, D49, D5, D50, D51, D52, D53, D54, D55, D56, D57, D58, D59, D6, D60, D61, D62, D63, D64, D65, D66, D67, D68, D69, D7, D70, D8, D9: D_Small, Diode_SMD:D_SOD-123, symbol Device:D_Small
- added MX_LALT2, MX_LCTRL2, MX_RCTRL2, MX_RMENU2: MX-LED, MX_Only:MXOnly-1.5U-FLIPPED, symbol MX_Alps_Hybrid:MX-LED
- added MX_LMENU2, MX_RMENU3, MX_RWIN2: MX-LED, MX_Only:MXOnly-1U-FLIPPED, symbol MX_Alps_Hybrid:MX-LED
- added MX_LSHFT2: MX-LED, MX_Only:MXOnly-1.25U-FLIPPED, symbol MX_Alps_Hybrid:MX-LED
- added MX_RCTRL3, MX_UP2: MX-LED, MX_Only:MXOnly-1U, symbol MX_Alps_Hybrid:MX-LED
- added MX_RSHFT2: MX-LED, MX_Only:MXOnly-1.75U-FLIPPED, symbol MX_Alps_Hybrid:MX-LED
- added MX_SPACE2: MX-LED, MX_Only:MXOnly-7U-FLIPPED-ReversedStabilizers, symbol MX_Alps_Hybrid:MX-LED
- MX_BSPC1: renamed from MX61; footprint MX_Only:MXOnly-2U-FLIPPED-ReversedStabilizers -> MX_Only:MXOnly-2U-FLIPPED
- MX_RCTRL1: renamed from MX60; footprint MX_Only:MXOnly-1U -> MX_Only:MXOnly-1.25U-FLIPPED
- SW2: footprint Pikatea Macropad Encoder Side Mount:Encoder-BI_EN11_HSM0E -> Pikatea:Encoder-BI_EN11_HSM0E
- renumbered MX45 to MX_0, MX7 to MX_1, MX11 to MX_2, MX16 to MX_3, MX20 to MX_4, MX24 to MX_5, MX28 to MX_6, MX33 to MX_7, MX37 to MX_8, MX41 to MX_9, MX42 to MX_<1, MX46 to MX_>1, MX10 to MX_A1, MX29 to MX_B1, MX62 to MX_BSLSH1, MX21 to MX_C1, MX4 to MX_CAPS1, MX58 to MX_CLBRK1, MX19 to MX_D1, MX64 to MX_DOWN1, MX18 to MX_E1, MX59 to MX_ENTER1, MX2 to MX_ESC1, MX8 to MX_EXTRA1, MX23 to MX_F1, MX51 to MX_FSLSH1, MX27 to MX_G1, MX32 to MX_H1, MX39 to MX_I1, MX36 to MX_J1, MX40 to MX_K1, MX44 to MX_L1, MX12 to MX_LALT1, MX1 to MX_LCTRL1, MX6 to MX_LMENU1, MX5 to MX_LSHFT1, MX38 to MX_M1, MX65 to MX_MACRO1, MX68 to MX_MACRO2, MX69 to MX_MACRO3, MX50 to MX_MINUS1, MX34 to MX_N1, MX43 to MX_O1, MX53 to MX_OPBRK1, MX48 to MX_P1, MX55 to MX_PLUS1, MX9 to MX_Q1, MX54 to MX_QUOTE1, MX22 to MX_R1, MX47 to MX_RALT1, MX67 to MX_RIGHT1, MX57 to MX_RMENU1, MX63 to MX_RSHFT1, MX52 to MX_RWIN1, MX15 to MX_S1, MX49 to MX_SEMI1, MX31 to MX_SPACE1, MX26 to MX_T1, MX3 to MX_TAB1, MX35 to MX_U1, MX66 to MX_UP1, MX25 to MX_V1, MX14 to MX_W1, MX17 to MX_X1, MX30 to MX_Y1, MX13 to MX_Z1
Connections:
- net D12 is gone; now on net Col4: U1.26 ((T1/~OC4D~/ADC9)PD6)
- net D6 is gone; now on net Col5: U1.27 ((T0/OC4D/ADC10)PD7)
- net D3: no longer U1.18 ((OC0B/SCL/INT0)PD0)
- net D4: no longer U1.25 ((ICP2/ADC8)PD4)
- net Col16: now reaches MX_CAPS1.1 (COL), MX_ESC1.1 (COL), MX_LCTRL1.1 (COL), MX_LSHFT1.1 (COL), MX_TAB1.1 (COL)
- net Col16: now also MX_LCTRL2.1 (COL), MX_LSHFT2.1 (COL)
- net Col15: now reaches MX_1.1 (COL), MX_A1.1 (COL), MX_EXTRA1.1 (COL), MX_LMENU1.1 (COL), MX_Q1.1 (COL)
- net Col15: now also MX_LMENU2.1 (COL)
- net Col14: now reaches MX_2.1 (COL), MX_LALT1.1 (COL), MX_S1.1 (COL), MX_W1.1 (COL), MX_Z1.1 (COL)
- net Col14: now also MX_LALT2.1 (COL)
- net Col13: now reaches MX_3.1 (COL), MX_D1.1 (COL), MX_E1.1 (COL), MX_X1.1 (COL)
- net Col12: now reaches MX_4.1 (COL), MX_C1.1 (COL), MX_F1.1 (COL), MX_R1.1 (COL)
- net Col11: now reaches MX_5.1 (COL), MX_G1.1 (COL), MX_T1.1 (COL), MX_V1.1 (COL)
- net Col10: now reaches MX_6.1 (COL), MX_B1.1 (COL), MX_H1.1 (COL), MX_SPACE1.1 (COL), MX_Y1.1 (COL)
- net Col10: now also MX_SPACE2.1 (COL)
- net Col9: now reaches MX_7.1 (COL), MX_J1.1 (COL), MX_N1.1 (COL), MX_U1.1 (COL)
- net Col8: now reaches MX_8.1 (COL), MX_I1.1 (COL), MX_K1.1 (COL), MX_M1.1 (COL)
- net Col7: now reaches MX_O1.1 (COL)
- net Col7: now also MX_9.1 (COL), MX_<1.1 (COL), MX_L1.1 (COL)
- net Col6: now reaches MX_0.1 (COL), MX_>1.1 (COL), MX_P1.1 (COL), MX_RALT1.1 (COL), MX_SEMI1.1 (COL)
- net Col5: now reaches MX_FSLSH1.1 (COL), MX_MINUS1.1 (COL), MX_OPBRK1.1 (COL), MX_QUOTE1.1 (COL), MX_RWIN1.1 (COL)
- net Col5: now also MX_RWIN2.1 (COL)
- net Col4: now reaches MX_CLBRK1.1 (COL), MX_PLUS1.1 (COL), MX_RMENU1.1 (COL)
- net Col4: now also MX_RMENU2.1 (COL), MX_RMENU3.1 (COL), MX_RSHFT2.1 (COL)
- net Col3: now reaches MX_BSLSH1.1 (COL), MX_BSPC1.1 (COL), MX_ENTER1.1 (COL), MX_RCTRL1.1 (COL), MX_RSHFT1.1 (COL)
- net Col3: now also U1.25 ((ICP2/ADC8)PD4), MX_RCTRL2.1 (COL), MX_RCTRL3.1 (COL), MX_UP2.1 (COL)
- net at MX_S1.2 (ROW): now also D12.2 (A)
- net at MX_D1.2 (ROW): now also D15.2 (A)
- net at MX_F1.2 (ROW): now also D18.2 (A)
- net at MX_G1.2 (ROW): now also D21.2 (A)
- net at MX_H1.2 (ROW): now also D25.2 (A)
- net at MX_J1.2 (ROW): now also D28.2 (A)
- net at MX_K1.2 (ROW): now also D31.2 (A)
- net at MX_L1.2 (ROW): now also D34.2 (A)
- net at MX_SEMI1.2 (ROW): now also D38.2 (A)
- net at MX_QUOTE1.2 (ROW): now also D42.2 (A)
- net COL2: now reaches MX_DOWN1.1 (COL), MX_MACRO1.1 (COL), MX_UP1.1 (COL)
- net COL2: now also SW2.S2
- net at MX_RSHFT1.3 (LED): now also MX_UP2.3 (LED)
- net at MX_RSHFT1.4 (LEDGND): now also MX_UP2.4 (LEDGND)
- net at MX_LCTRL1.3 (LED): now also MX_LCTRL2.3 (LED)
- net at MX_LCTRL1.4 (LEDGND): now also MX_LCTRL2.4 (LEDGND)
- net at MX_LMENU1.3 (LED): now also MX_LMENU2.3 (LED)
- net at MX_LMENU1.4 (LEDGND): now also MX_LMENU2.4 (LEDGND)
- net at MX_LALT1.3 (LED): now also MX_LALT2.3 (LED)
- net at MX_LALT1.4 (LEDGND): now also MX_LALT2.4 (LEDGND)
- net at MX_SPACE1.3 (LED): now also MX_SPACE2.3 (LED)
- net at MX_SPACE1.4 (LEDGND): now also MX_SPACE2.4 (LEDGND)
- net at MX_RWIN1.3 (LED): now also MX_RWIN2.3 (LED)
- net at MX_RWIN1.4 (LEDGND): now also MX_RWIN2.4 (LEDGND)
- net at MX_RMENU1.3 (LED): now also MX_RMENU2.3 (LED), MX_RMENU3.3 (LED)
- net at MX_RMENU1.4 (LEDGND): now also MX_RMENU2.4 (LEDGND), MX_RMENU3.4 (LEDGND)
- net at MX_RCTRL1.3 (LED): now also MX_RCTRL2.3 (LED), MX_RCTRL3.3 (LED)
- net at MX_RCTRL1.4 (LEDGND): now also MX_RCTRL2.4 (LEDGND), MX_RCTRL3.4 (LEDGND)
- net at MX_A1.2 (ROW): now also D8.2 (A)
- net A0: no longer names the net of U1.36 ((ADC7/TDI)PF7)
- net A0: no longer SW2.S2
- net CS: no longer names the net of U1.30 ((ADC13/OC1B/OC4B/PCINT13)PB6)
- net D0: no longer names the net of U1.41 ((ADC0)PF0)
- net D1: no longer names the net of U1.40 ((ADC1)PF1)
- net D11: no longer names the net of U1.12 ((OC0A/OC1C/~RTS~/PCINT7)PB7)
- net D13: no longer names the net of U1.32 ((ICP3/CLK0/OC4A)PC7)
- net D2: no longer names the net of U1.19 ((SDA/INT1)PD1)
- net D2: no longer SW2.S1
- net D5: no longer names the net of U1.31 ((OC3A/~OC4A~)PC6)
- net D7: no longer names the net of U1.1 ((INT6/AIN0)PE6)
- net D8: no longer names the net of U1.28 ((ADC11/PCINT4)PB4)
- net D9: no longer names the net of U1.29 ((ADC12/OC1A/~OC4B~/PCINT12)PB5)
- new net: D69.2 (A), SW2.S1
- new net: D2.2 (A), MX_TAB1.2 (ROW)
- new net: D7.2 (A), MX_Q1.2 (ROW)
- new net: D11.2 (A), MX_W1.2 (ROW)
- new net: D14.2 (A), MX_E1.2 (ROW)
- new net: D17.2 (A), MX_R1.2 (ROW)
- new net: D20.2 (A), MX_T1.2 (ROW)
- new net: D23.2 (A), MX_Y1.2 (ROW)
- new net: D27.2 (A), MX_U1.2 (ROW)
- new net: D30.2 (A), MX_I1.2 (ROW)
- new net: D33.2 (A), MX_O1.2 (ROW)
- new net: D37.2 (A), MX_P1.2 (ROW)
- new net: D41.2 (A), MX_OPBRK1.2 (ROW)
- new net: D44.2 (A), MX_CLBRK1.2 (ROW)
- new net: D47.2 (A), MX_BSLSH1.2 (ROW)
- new net: D3.2 (A), MX_CAPS1.2 (ROW)
- new net: D45.2 (A), MX_ENTER1.2 (ROW)
- new net: D50.2 (A), MX_MACRO1.2 (ROW)
- new net: D53.2 (A), MX_MACRO2.2 (ROW)
- new net: D4.2 (A), MX_LSHFT1.2 (ROW), MX_LSHFT2.2 (ROW)
- new net: D10.2 (A), MX_Z1.2 (ROW)
- new net: D13.2 (A), MX_X1.2 (ROW)
- new net: D16.2 (A), MX_C1.2 (ROW)
- new net: D19.2 (A), MX_V1.2 (ROW)
- new net: D22.2 (A), MX_B1.2 (ROW)
- new net: D26.2 (A), MX_N1.2 (ROW)
- new net: D29.2 (A), MX_M1.2 (ROW)
- new net: D32.2 (A), MX_<1.2 (ROW)
- new net: D35.2 (A), MX_>1.2 (ROW)
- new net: D39.2 (A), MX_FSLSH1.2 (ROW)
- new net: D48.2 (A), MX_RSHFT1.2 (ROW), MX_UP2.2 (ROW)
- new net: D51.2 (A), MX_UP1.2 (ROW)
- new net: D1.2 (A), MX_LCTRL1.2 (ROW), MX_LCTRL2.2 (ROW)
- new net: D5.2 (A), MX_LMENU1.2 (ROW), MX_LMENU2.2 (ROW)
- new net: D9.2 (A), MX_LALT1.2 (ROW), MX_LALT2.2 (ROW)
- new net: D24.2 (A), MX_SPACE1.2 (ROW), MX_SPACE2.2 (ROW)
- new net: D36.2 (A), MX_RALT1.2 (ROW)
- new net: D40.2 (A), MX_RWIN1.2 (ROW), MX_RWIN2.2 (ROW)
- new net: D43.2 (A), MX_RMENU1.2 (ROW), MX_RMENU2.2 (ROW), MX_RMENU3.2 (ROW)
- new net: D46.2 (A), MX_RCTRL1.2 (ROW), MX_RCTRL2.2 (ROW), MX_RCTRL3.2 (ROW)
- new net: D49.2 (A), MX_DOWN1.2 (ROW)
- new net: D52.2 (A), MX_RIGHT1.2 (ROW)
- new net: D54.2 (A), MX_MACRO3.2 (ROW)
- new net: D55.2 (A), MX_ESC1.2 (ROW)
- new net: D56.2 (A), MX_1.2 (ROW)
- new net: D57.2 (A), MX_2.2 (ROW)
- new net: D58.2 (A), MX_3.2 (ROW)
- new net: D59.2 (A), MX_4.2 (ROW)
- new net: D60.2 (A), MX_5.2 (ROW)
- new net: D61.2 (A), MX_6.2 (ROW)
- new net: D62.2 (A), MX_7.2 (ROW)
- new net: D63.2 (A), MX_8.2 (ROW)
- new net: D64.2 (A), MX_9.2 (ROW)
- new net: D65.2 (A), MX_0.2 (ROW)
- new net: D66.2 (A), MX_MINUS1.2 (ROW)
- new net: D67.2 (A), MX_PLUS1.2 (ROW)
- new net: D68.2 (A), MX_BSPC1.2 (ROW)
- new net: D6.2 (A), MX_EXTRA1.2 (ROW)
- new net: D70.2 (A), MX_RSHFT2.2 (ROW)
- new net Row1: D55.1 (K), D56.1 (K), D57.1 (K), D58.1 (K), D59.1 (K), D60.1 (K), D61.1 (K), D62.1 (K), D63.1 (K), D64.1 (K), D65.1 (K), D66.1 (K), D67.1 (K), D68.1 (K), D69.1 (K)
- new net Row2: D11.1 (K), D14.1 (K), D17.1 (K), D2.1 (K), D20.1 (K), D23.1 (K), D27.1 (K), D30.1 (K), D33.1 (K), D37.1 (K), D41.1 (K), D44.1 (K), D47.1 (K), D7.1 (K)
- new net Row3: D12.1 (K), D15.1 (K), D18.1 (K), D21.1 (K), D25.1 (K), D28.1 (K), D3.1 (K), D31.1 (K), D34.1 (K), D38.1 (K), D42.1 (K), D45.1 (K), D50.1 (K), D53.1 (K), D8.1 (K)
- new net Row4: D10.1 (K), D13.1 (K), D16.1 (K), D19.1 (K), D22.1 (K), D26.1 (K), D29.1 (K), D32.1 (K), D35.1 (K), D39.1 (K), D4.1 (K), D48.1 (K), D51.1 (K), D54.1 (K), D6.1 (K), D70.1 (K)
- new net Row5: D1.1 (K), D24.1 (K), D36.1 (K), D40.1 (K), D43.1 (K), D46.1 (K), D49.1 (K), D5.1 (K), D52.1 (K), D9.1 (K)
Other:
- moved on the sheet: MX_0, MX_1, MX_2, MX_3, MX_4, MX_5, MX_6, MX_7, MX_8, MX_9, MX_<1, MX_>1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
