File: Pikatea Keyboard/Pikatea Keyboard.kicad_pcb (KiCad board)
At the start: 2 copper layers, 319.6 x 93.7 mm, 87 parts, among them J1 AVR-ISP-6, J2 USB_B_Mini, SW1 SW_DPST, SW2 Rotary_Encoder_Switch, U1 ATMEGA32U4-EP, X1 16MHz

Commit message: update keyboard
Parts:
- removed MX31: MX-LED, MX_Only:MXOnly-6.25U-FLIPPED-ReversedStabilizers
- removed MX6: MX-LED, MX_Only:MXOnly-1.25U-FLIPPED
- removed MX65, MX68: MX-LED, MX_Only:MXOnly-1U
- added D1: D_Small, Diode_SMD:D_SOD-123, F.Cu at (260.6, 142.9)
- added D10: D_Small, Diode_SMD:D_SOD-123, F.Cu at (222.7, 124.4)
- added D11: D_Small, Diode_SMD:D_SOD-123, F.Cu at (216.2, 92.9)
- added D12: D_Small, Diode_SMD:D_SOD-123, F.Cu at (213.5, 105.3)
- added D13: D_Small, Diode_SMD:D_SOD-123, F.Cu at (203.6, 124.4)
- added D14: D_Small, Diode_SMD:D_SOD-123, F.Cu at (197.2, 92.8)
- added D15: D_Small, Diode_SMD:D_SOD-123, F.Cu at (191.9, 105.5)
- added D16: D_Small, Diode_SMD:D_SOD-123, F.Cu at (183.7, 124.2)
- added D17: D_Small, Diode_SMD:D_SOD-123, F.Cu at (177.9, 92.6)
- added D18: D_Small, Diode_SMD:D_SOD-123, F.Cu at (174.4, 105.3)
- added D19: D_Small, Diode_SMD:D_SOD-123, F.Cu at (165.5, 124.6)
- added D2: D_Small, Diode_SMD:D_SOD-123, F.Cu at (259.1, 92.6)
- added D20: D_Small, Diode_SMD:D_SOD-123, F.Cu at (159.0, 92.9)
- added D21: D_Small, Diode_SMD:D_SOD-123, F.Cu at (154.7, 105.2)
- added D22: D_Small, Diode_SMD:D_SOD-123, F.Cu at (145.9, 124.3)
- added D23: D_Small, Diode_SMD:D_SOD-123, F.Cu at (140.0, 92.8)
- added D24: D_Small, Diode_SMD:D_SOD-123, F.Cu at (144.0, 143.4)
- added D25: D_Small, Diode_SMD:D_SOD-123, F.Cu at (136.7, 105.3)
- added D26: D_Small, Diode_SMD:D_SOD-123, F.Cu at (127.1, 124.2)
- added D27: D_Small, Diode_SMD:D_SOD-123, F.Cu at (121.0, 93.0)
- added D28: D_Small, Diode_SMD:D_SOD-123, F.Cu at (117.8, 105.5)
- added D29: D_Small, Diode_SMD:D_SOD-123, F.Cu at (107.2, 124.2)
- added D3: D_Small, Diode_SMD:D_SOD-123, F.Cu at (257.9, 105.0)
- added D30: D_Small, Diode_SMD:D_SOD-123, F.Cu at (101.8, 93.0)
- added D31: D_Small, Diode_SMD:D_SOD-123, F.Cu at (98.8, 105.5)
- added D32: D_Small, Diode_SMD:D_SOD-123, F.Cu at (88.6, 124.5)
- added D33: D_Small, Diode_SMD:D_SOD-123, F.Cu at (82.7, 92.9)
- added D34: D_Small, Diode_SMD:D_SOD-123, F.Cu at (79.8, 105.2)
- added D35: D_Small, Diode_SMD:D_SOD-123, F.Cu at (69.2, 124.3)
- added D36: D_Small, Diode_SMD:D_SOD-123, F.Cu at (71.2, 143.6)
- added D37: D_Small, Diode_SMD:D_SOD-123, F.Cu at (63.6, 92.7)
- added D38: D_Small, Diode_SMD:D_SOD-123, F.Cu at (60.2, 105.1)
- added D39: D_Small, Diode_SMD:D_SOD-123, F.Cu at (50.3, 124.3)
- added D4: D_Small, Diode_SMD:D_SOD-123, F.Cu at (262.0, 124.2)
- added D40: D_Small, Diode_SMD:D_SOD-123, F.Cu at (48.3, 143.6)
- added D41: D_Small, Diode_SMD:D_SOD-123, F.Cu at (44.8, 89.5)
- added D42: D_Small, Diode_SMD:D_SOD-123, F.Cu at (41.7, 105.2)
- added D43: D_Small, Diode_SMD:D_SOD-123, F.Cu at (24.4, 143.6)
- added D44: D_Small, Diode_SMD:D_SOD-123, F.Cu at (25.7, 90.2)
- added D45: D_Small, Diode_SMD:D_SOD-123, F.Cu at (10.9, 105.7)
- added D46: D_Small, Diode_SMD:D_SOD-123, F.Cu at (-1.25, 143.6)
- added D47: D_Small, Diode_SMD:D_SOD-123, F.Cu at (15.7, 96.3)
- added D48: D_Small, Diode_SMD:D_SOD-123, F.Cu at (14.8, 124.4)
- added D49: D_Small, Diode_SMD:D_SOD-123, F.Cu at (-21.1, 143.2)
- added D5: D_Small, Diode_SMD:D_SOD-123, F.Cu at (236.5, 143.0)
- added D50: D_Small, Diode_SMD:D_SOD-123, F.Cu at (-21.1, 118.6)
- added D51: D_Small, Diode_SMD:D_SOD-123, F.Cu at (-20.7, 124.2)
- added D52: D_Small, Diode_SMD:D_SOD-123, F.Cu at (-33.3, 142.1)
- added D53: D_Small, Diode_SMD:D_SOD-123, F.Cu at (-38.1, 118.4)
- added D54: D_Small, Diode_SMD:D_SOD-123, F.Cu at (-32.4, 122.7)
- added D55: D_Small, Diode_SMD:D_SOD-123, F.Cu at (260.3, 68.0)
- added D56: D_Small, Diode_SMD:D_SOD-123, F.Cu at (253.1, 68.0)
- added D57: D_Small, Diode_SMD:D_SOD-123, F.Cu at (225.9, 68.7)
- added D58: D_Small, Diode_SMD:D_SOD-123, F.Cu at (207.3, 68.9)
- added D59: D_Small, Diode_SMD:D_SOD-123, F.Cu at (188.7, 68.5)
- added D6: D_Small, Diode_SMD:D_SOD-123, F.Cu at (240.8, 124.3)
- added D60: D_Small, Diode_SMD:D_SOD-123, F.Cu at (169.5, 68.4)
- added D61: D_Small, Diode_SMD:D_SOD-123, F.Cu at (150.5, 68.5)
- added D62: D_Small, Diode_SMD:D_SOD-123, F.Cu at (130.9, 68.8)
- added D63: D_Small, Diode_SMD:D_SOD-123, F.Cu at (112.1, 69.0)
- added D64: D_Small, Diode_SMD:D_SOD-123, F.Cu at (92.4, 68.5)
- added D65: D_Small, Diode_SMD:D_SOD-123, F.Cu at (73.6, 68.9)
- added D66: D_Small, Diode_SMD:D_SOD-123, F.Cu at (54.6, 68.8)
- added D67: D_Small, Diode_SMD:D_SOD-123, F.Cu at (36.0, 69.0)
- added D68: D_Small, Diode_SMD:D_SOD-123, F.Cu at (7.32, 68.7)
- added D69: D_Small, Diode_SMD:D_SOD-123, F.Cu at (-14.7, 72.9)
- added D7: D_Small, Diode_SMD:D_SOD-123, F.Cu at (235.4, 92.7)
- added D70: D_Small, Diode_SMD:D_SOD-123, F.Cu at (25.0, 124.3)
- added D8: D_Small, Diode_SMD:D_SOD-123, F.Cu at (232.0, 105.2)
- added D9: D_Small, Diode_SMD:D_SOD-123, F.Cu at (212.5, 143.1)
- added MX_LALT2: MX-LED, MX_Only:MXOnly-1.5U-FLIPPED, B.Cu at (219.1, 150.0)
- added MX_LCTRL2: MX-LED, MX_Only:MXOnly-1.5U-FLIPPED, B.Cu at (266.7, 150.0)
- added MX_LMENU1: MX-LED, MX_Only:MXOnly-1.25U-FLIPPED, B.Cu at (245.2, 150.0)
- added MX_LMENU2: MX-LED, MX_Only:MXOnly-1U-FLIPPED, B.Cu at (242.9, 150.0)
- added MX_LSHFT2: MX-LED, MX_Only:MXOnly-1.25U-FLIPPED, B.Cu at (269.1, 130.9)
- added MX_MACRO1: MX-LED, MX_Only:MXOnly-1U, B.Cu at (-14.3, 111.9)
- added MX_MACRO2: MX-LED, MX_Only:MXOnly-1U, B.Cu at (-33.3, 111.9)
- added MX_RCTRL2: MX-LED, MX_Only:MXOnly-1.5U-FLIPPED, B.Cu at (9.52, 150.0)
- added MX_RCTRL3: MX-LED, MX_Only:MXOnly-1U, B.Cu at (4.76, 150.0)
- added MX_RMENU2: MX-LED, MX_Only:MXOnly-1.5U-FLIPPED, F.Cu at (38.1, 150.0)
- added MX_RMENU3: MX-LED, MX_Only:MXOnly-1U-FLIPPED, B.Cu at (23.8, 150.0)
- added MX_RSHFT2: MX-LED, MX_Only:MXOnly-1.75U-FLIPPED, B.Cu at (31.0, 130.9)
- added MX_RWIN2: MX-LED, MX_Only:MXOnly-1U-FLIPPED, B.Cu at (61.9, 150.0)
- added MX_SPACE1: MX-LED, MX_Only:MXOnly-6.25U-FLIPPED-ReversedStabilizers, B.Cu at (150.0, 150.0)
- added MX_SPACE2: MX-LED, MX_Only:MXOnly-7U-FLIPPED-ReversedStabilizers, B.Cu at (138.1, 150.0)
- added MX_UP2: MX-LED, MX_Only:MXOnly-1U, F.Cu at (4.76, 130.9)
- MX_RCTRL1: renamed from MX60; footprint MX_Only:MXOnly-1U -> MX_Only:MXOnly-1.25U-FLIPPED
- SW2: footprint Pikatea Macropad Encoder Side Mount:Encoder-BI_EN11_HSM0E -> Pikatea:Encoder-BI_EN11_HSM0E
- moved R4 236.8 mm to (-31.9, 92.5)
- moved R5 233.2 mm to (-31.9, 90.0)
- moved C4 229.3 mm to (-20.1, 93.2), turned to 45 degrees
- moved C2 224.7 mm to (-14.3, 86.3), turned to 225 degrees
- moved C5 213.9 mm to (-18.9, 99.9), turned to 135 degrees
- moved C3 213.3 mm to (0.42, 92.0), turned to 315 degrees
- moved X1 190.6 mm to (-0.81, 104.8), turned to 180 degrees
- moved U1 188.5 mm to (-9.28, 96.6), turned to 45 degrees
- moved C6 166.9 mm to (-24.2, 93.6), turned to 270 degrees
- moved J1 163.5 mm to (-36.8, 97.6), turned to 90 degrees
- moved C10 154.3 mm to (-17.6, 91.5), turned to 135 degrees
- moved C9 149.4 mm to (-16.0, 104.0), turned to 135 degrees
- moved R3 145.0 mm to (-9.72, 106.6)
- moved C8 140.7 mm to (-4.03, 105.8), turned to 270 degrees
- moved C7 138.6 mm to (0.66, 102.1)
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- renumbered MX45 to MX_0, MX7 to MX_1, MX11 to MX_2, MX16 to MX_3, MX20 to MX_4, MX24 to MX_5, MX28 to MX_6, MX33 to MX_7, MX37 to MX_8, MX41 to MX_9, MX42 to MX_<1, MX46 to MX_>1, MX10 to MX_A1, MX29 to MX_B1, MX62 to MX_BSLSH1, MX61 to MX_BSPC1, MX21 to MX_C1, MX4 to MX_CAPS1, MX58 to MX_CLBRK1, MX19 to MX_D1, MX64 to MX_DOWN1, MX18 to MX_E1, MX59 to MX_ENTER1, MX2 to MX_ESC1, MX8 to MX_EXTRA1, MX23 to MX_F1, MX51 to MX_FSLSH1, MX27 to MX_G1, MX32 to MX_H1, MX39 to MX_I1, MX36 to MX_J1, MX40 to MX_K1, MX44 to MX_L1, MX12 to MX_LALT1, MX1 to MX_LCTRL1, MX5 to MX_LSHFT1, MX38 to MX_M1, MX69 to MX_MACRO3, MX50 to MX_MINUS1, MX34 to MX_N1, MX43 to MX_O1, MX53 to MX_OPBRK1, MX48 to MX_P1, MX55 to MX_PLUS1, MX9 to MX_Q1, MX54 to MX_QUOTE1, MX22 to MX_R1, MX47 to MX_RALT1, MX67 to MX_RIGHT1, MX57 to MX_RMENU1, MX63 to MX_RSHFT1, MX52 to MX_RWIN1, MX15 to MX_S1, MX49 to MX_SEMI1, MX26 to MX_T1, MX3 to MX_TAB1, MX35 to MX_U1, MX66 to MX_UP1, MX25 to MX_V1, MX14 to MX_W1, MX17 to MX_X1, MX30 to MX_Y1, MX13 to MX_Z1
Connections:
- net /CS renamed Net-(U1-Pad30)
- net /D0 renamed Net-(U1-Pad41)
- net /D1 renamed Net-(U1-Pad40)
- net /D11 renamed Net-(U1-Pad12)
- net /D13 renamed Net-(U1-Pad32)
- net /D5 renamed Net-(U1-Pad31)
- net /D7 renamed Net-(U1-Pad1)
- net /D8 renamed Net-(U1-Pad28)
- net /D9 renamed Net-(U1-Pad29)
- net Net-(MX1-Pad1) renamed Col16
- net Net-(MX10-Pad1) renamed Col15
- net Net-(MX11-Pad1) renamed Col14
- net Net-(MX16-Pad1) renamed Col13
- net Net-(MX20-Pad1) renamed Col12
- net Net-(MX24-Pad1) renamed Col11
- net Net-(MX28-Pad1) renamed Col10
- net Net-(MX33-Pad1) renamed Col9
- net Net-(MX37-Pad1) renamed Col8
- net Net-(MX45-Pad1) renamed Col6
- MX_0 pad 2: Net-(MX11-Pad2) -> Net-(D65-Pad2)
- MX_1 pad 2: Net-(MX11-Pad2) -> Net-(D56-Pad2)
- MX_2 pad 2: Net-(MX11-Pad2) -> Net-(D57-Pad2)
- MX_3 pad 2: Net-(MX11-Pad2) -> Net-(D58-Pad2)
- MX_4 pad 2: Net-(MX11-Pad2) -> Net-(D59-Pad2)
- MX_5 pad 2: Net-(MX11-Pad2) -> Net-(D60-Pad2)
- MX_6 pad 2: Net-(MX11-Pad2) -> Net-(D61-Pad2)
- MX_7 pad 2: Net-(MX11-Pad2) -> Net-(D62-Pad2)
- MX_8 pad 2: Net-(MX11-Pad2) -> Net-(D63-Pad2)
- MX_9 pad 1: Net-(MX41-Pad1) -> Col7
- MX_9 pad 2: Net-(MX11-Pad2) -> Net-(D64-Pad2)
- MX_<1 pad 1: Net-(MX41-Pad1) -> Col7
- MX_<1 pad 2: Net-(MX13-Pad2) -> Net-(D32-Pad2)
- MX_>1 pad 2: Net-(MX13-Pad2) -> Net-(D35-Pad2)
- MX_B1 pad 2: Net-(MX13-Pad2) -> Net-(D22-Pad2)
- MX_BSLSH1 pad 1: Net-(MX59-Pad1) -> Col3
- MX_BSLSH1 pad 2: Net-(MX14-Pad2) -> Net-(D47-Pad2)
- MX_BSPC1 pad 1: Net-(MX59-Pad1) -> Col3
- MX_BSPC1 pad 2: Net-(MX11-Pad2) -> Net-(D68-Pad2)
- MX_C1 pad 2: Net-(MX13-Pad2) -> Net-(D16-Pad2)
- MX_CAPS1 pad 2: Net-(MX4-Pad2) -> Net-(D3-Pad2)
- MX_CLBRK1 pad 1: Net-(MX55-Pad1) -> Col4
- MX_CLBRK1 pad 2: Net-(MX14-Pad2) -> Net-(D44-Pad2)
- MX_DOWN1 pad 1: Net-(MX64-Pad1) -> COL2
- MX_DOWN1 pad 2: Net-(MX1-Pad2) -> Net-(D49-Pad2)
- MX_E1 pad 2: Net-(MX14-Pad2) -> Net-(D14-Pad2)
- MX_ENTER1 pad 1: Net-(MX59-Pad1) -> Col3
- MX_ENTER1 pad 2: Net-(MX4-Pad2) -> Net-(D45-Pad2)
- MX_ESC1 pad 2: Net-(MX11-Pad2) -> Net-(D55-Pad2)
- MX_EXTRA1 pad 2: Net-(MX13-Pad2) -> Net-(D6-Pad2)
- MX_FSLSH1 pad 1: Net-(MX50-Pad1) -> Col5
- MX_FSLSH1 pad 2: Net-(MX13-Pad2) -> Net-(D39-Pad2)
- MX_I1 pad 2: Net-(MX14-Pad2) -> Net-(D30-Pad2)
- MX_L1 pad 1: Net-(MX41-Pad1) -> Col7
- MX_LALT1 pad 2: Net-(MX1-Pad2) -> Net-(D9-Pad2)
- MX_LCTRL1 pad 2: Net-(MX1-Pad2) -> Net-(D1-Pad2)
- MX_LSHFT1 pad 2: Net-(MX13-Pad2) -> Net-(D4-Pad2)
- MX_M1 pad 2: Net-(MX13-Pad2) -> Net-(D29-Pad2)
- MX_MACRO3 pad 2: Net-(MX13-Pad2) -> Net-(D54-Pad2)
- MX_MINUS1 pad 1: Net-(MX50-Pad1) -> Col5
- MX_MINUS1 pad 2: Net-(MX11-Pad2) -> Net-(D66-Pad2)
- MX_N1 pad 2: Net-(MX13-Pad2) -> Net-(D26-Pad2)
- MX_O1 pad 1: Net-(MX43-Pad1) -> Col7
- MX_O1 pad 2: Net-(MX14-Pad2) -> Net-(D33-Pad2)
- MX_OPBRK1 pad 1: Net-(MX50-Pad1) -> Col5
- MX_OPBRK1 pad 2: Net-(MX14-Pad2) -> Net-(D41-Pad2)
- MX_P1 pad 2: Net-(MX14-Pad2) -> Net-(D37-Pad2)
- MX_PLUS1 pad 1: Net-(MX55-Pad1) -> Col4
- MX_PLUS1 pad 2: Net-(MX11-Pad2) -> Net-(D67-Pad2)
- MX_Q1 pad 2: Net-(MX14-Pad2) -> Net-(D7-Pad2)
- MX_QUOTE1 pad 1: Net-(MX50-Pad1) -> Col5
- MX_R1 pad 2: Net-(MX14-Pad2) -> Net-(D17-Pad2)
- MX_RALT1 pad 2: Net-(MX1-Pad2) -> Net-(D36-Pad2)
- MX_RCTRL1 pad 1: Net-(MX59-Pad1) -> Col3
- MX_RCTRL1 pad 2: Net-(MX1-Pad2) -> Net-(D46-Pad2)
- MX_RIGHT1 pad 2: Net-(MX1-Pad2) -> Net-(D52-Pad2)
- MX_RMENU1 pad 1: Net-(MX55-Pad1) -> Col4
- MX_RMENU1 pad 2: Net-(MX1-Pad2) -> Net-(D43-Pad2)
- MX_RSHFT1 pad 1: Net-(MX59-Pad1) -> Col3
- MX_RSHFT1 pad 2: Net-(MX13-Pad2) -> Net-(D48-Pad2)
- MX_RWIN1 pad 1: Net-(MX50-Pad1) -> Col5
- MX_RWIN1 pad 2: Net-(MX1-Pad2) -> Net-(D40-Pad2)
- MX_T1 pad 2: Net-(MX14-Pad2) -> Net-(D20-Pad2)
- MX_TAB1 pad 2: Net-(MX14-Pad2) -> Net-(D2-Pad2)
- MX_U1 pad 2: Net-(MX14-Pad2) -> Net-(D27-Pad2)
- MX_UP1 pad 1: Net-(MX64-Pad1) -> COL2
- MX_UP1 pad 2: Net-(MX13-Pad2) -> Net-(D51-Pad2)
- MX_V1 pad 2: Net-(MX13-Pad2) -> Net-(D19-Pad2)
- MX_W1 pad 2: Net-(MX14-Pad2) -> Net-(D11-Pad2)
- MX_X1 pad 2: Net-(MX13-Pad2) -> Net-(D13-Pad2)
- MX_Y1 pad 2: Net-(MX14-Pad2) -> Net-(D23-Pad2)
- MX_Z1 pad 2: Net-(MX13-Pad2) -> Net-(D10-Pad2)
- SW2 pad S1: /D2 -> Net-(D69-Pad2)
- SW2 pad S2: /A0 -> COL2
- U1 pad 18: /D3 -> Net-(U1-Pad18)
- U1 pad 19: /D2 -> Net-(U1-Pad19)
- U1 pad 25: /D4 -> Col3
- U1 pad 26: /D12 -> Col4
- U1 pad 27: /D6 -> Col5
- U1 pad 36: /A0 -> Net-(U1-Pad36)
Routing:
- net VBUS: track 0.00 -> 422.7 mm, vias 0 -> 9
- net Row3: track 0.00 -> 317.6 mm
- net /D-: track 0.00 -> 310.3 mm
- net /D+: track 0.00 -> 309.7 mm
- net Row4: track 0.00 -> 299.2 mm
- net Row5: track 0.00 -> 296.7 mm
- net Row1: track 0.00 -> 281.7 mm
- net Row2: track 0.00 -> 256.3 mm
- net /RESET: track 0.00 -> 213.2 mm, vias 0 -> 4
- net Col5: track 0.00 -> 158.4 mm
- net Col3: track 0.00 -> 147.2 mm
- net Col4: track 0.00 -> 134.5 mm
- net Col10: track 0.00 -> 99.9 mm
- net Col16: track 0.00 -> 93.9 mm
- net Col14: track 0.00 -> 92.3 mm
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- added copper zone on B.Cu, net GND
- added copper zone on F.Cu, net GND
Other:
- outline, holes or cut-outs redrawn

Commit message: finish pcb shape and add holes for standoffs
Parts:
- moved D50 3.13 mm to (-21.1, 115.4)
- moved D51 2.42 mm to (-19.9, 126.5), turned to 90 degrees
Routing:
- net Net-(D50-Pad2): track 13.8 -> 4.62 mm
- net Row4: track 299.2 -> 304.2 mm
- net Row3: track 317.6 -> 320.1 mm
- net Net-(D46-Pad2): track 5.96 -> 8.34 mm
- net /D-: track 310.3 -> 311.7 mm
- net VBUS: track 422.7 -> 424.1 mm
- net /D+: track 309.7 -> 311.1 mm
- net Col10: track 99.9 -> 99.0 mm
- net Row2: track 256.3 -> 257.0 mm
Other:
- outline, holes or cut-outs redrawn
