File: Pikatea Keyboard ProMicro/Pikatea Keyboard Pro Micro.kicad_pcb (KiCad board)
At the start: 2 copper layers, 319.6 x 93.7 mm, 153 parts, among them SW2 Rotary_Encoder_Switch, U1 Teensy2.0_(Arduino), U2 Teensy2.0_(Arduino)

Commit message: updates
Connections:
- SW2 pad A: (no net) -> /D4
- SW2 pad B: (no net) -> /D3
- U1 pad 10: Net-(U1-Pad10) -> COL2
- U1 pad 11: Net-(U1-Pad11) -> Col3
- U1 pad 12: Net-(U1-Pad12) -> Col4
- U1 pad 13: Net-(U1-Pad13) -> Col5
- U1 pad 19: Net-(U1-Pad19) -> Col16
- U1 pad 2: Net-(U1-Pad2) -> Row1
- U1 pad 20: Net-(U1-Pad20) -> Col15
- U1 pad 21: Net-(U1-Pad21) -> Col14
- U1 pad 22: Net-(U1-Pad22) -> Col13
- U1 pad 23: Net-(U1-Pad23) -> Col12
- U1 pad 24: Net-(U1-Pad24) -> Col11
- U1 pad 25: Net-(U1-Pad25) -> Col10
- U1 pad 26: Net-(U1-Pad26) -> Col9
- U1 pad 27: Net-(U1-Pad27) -> Col8
- U1 pad 28: Net-(U1-Pad28) -> Col7
- U1 pad 3: Net-(U1-Pad3) -> Row2
- U1 pad 30: Net-(U1-Pad30) -> Col6
- U1 pad 4: Net-(U1-Pad4) -> Row3
- U1 pad 5: Net-(U1-Pad5) -> /D3
- U1 pad 6: Net-(U1-Pad6) -> /D4
- U1 pad 7: Net-(U1-Pad7) -> Row4
- U1 pad 8: Net-(U1-Pad8) -> Row5
- U1 pad 9: Net-(U1-Pad9) -> Col1
- U2 pad 10: Net-(U1-Pad10) -> COL2
- U2 pad 11: Net-(U1-Pad11) -> Col3
- U2 pad 12: Net-(U1-Pad12) -> Col4
- U2 pad 13: Net-(U1-Pad13) -> Col5
- U2 pad 19: Net-(U1-Pad19) -> Col16
- U2 pad 2: Net-(U1-Pad2) -> Row1
- U2 pad 20: Net-(U1-Pad20) -> Col15
- U2 pad 21: Net-(U1-Pad21) -> Col14
- U2 pad 22: Net-(U1-Pad22) -> Col13
- U2 pad 23: Net-(U1-Pad23) -> Col12
- U2 pad 24: Net-(U1-Pad24) -> Col11
- U2 pad 25: Net-(U1-Pad25) -> Col10
- U2 pad 26: Net-(U1-Pad26) -> Col9
- U2 pad 27: Net-(U1-Pad27) -> Col8
- U2 pad 28: Net-(U1-Pad28) -> Col7
- U2 pad 3: Net-(U1-Pad3) -> Row2
- U2 pad 30: Net-(U1-Pad30) -> Col6
- U2 pad 4: Net-(U1-Pad4) -> Row3
- U2 pad 5: Net-(U1-Pad5) -> /D3
- U2 pad 6: Net-(U1-Pad6) -> /D4
- U2 pad 7: Net-(U1-Pad7) -> Row4
- U2 pad 8: Net-(U1-Pad8) -> Row5
- U2 pad 9: Net-(U1-Pad9) -> Col1
