File: Pikatea Macropad GB3 Addon/Pikatea Macropad GB3 Addon.kicad_pcb (KiCad board)
At the start: 2 copper layers, 125.1 x 25.2 mm, 29 parts, among them J1 AVR-ISP-6, J2 USB_B_Mini, J3 Conn_01x03_Male, J4 Conn_01x03_Male, J5 Conn_01x03_Male, J6 Conn_01x06_Male, J7 Conn_01x03_Male, SW1 SW_DPST, SW2 Rotary_Encoder_Switch, U1 ATMEGA32U4-EP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

Commit message: add gb3 addon
Parts:
- removed C1, C10, C2, C3, C4, C5: 0u1, Capacitor_SMD:C_0805_2012Metric
- removed C6: 4u7, Capacitor_SMD:C_0805_2012Metric
- removed C7, C8: 22p, Capacitor_SMD:C_0805_2012Metric
- removed C9: 1u, Capacitor_SMD:C_0805_2012Metric
- removed J1: AVR-ISP-6, keyboard_parts:AVR_ICSP_3x2
- removed J2: USB_B_Mini, usb_mini:USB-Mini-B_ LCSC-C46398
- removed J3, J7: Conn_01x03_Male, Connector_PinHeader_2.54mm:PinHeader_1x03_P2.54mm_Vertical
- removed J6: Conn_01x06_Male, Pikatea Macropad Encoder Side Mount:Breakaway-Throughole
- removed MX1, MX2, MX3: MX-LED, MX_Only:MXOnly-1U
- removed R3: 10K, Resistor_SMD:R_0805_2012Metric
- removed R4, R5: 22, Resistor_SMD:R_0805_2012Metric
- removed SW1: SW_DPST, Button_Switch_SMD:SW_SPST_TL3342
- removed SW2: Rotary_Encoder_Switch, Pikatea Macropad Encoder Side Mount:Encoder-BI_EN11_HSM0E
- removed U1: ATMEGA32U4-EP, Package_QFP:LQFP-44_10x10mm_P0.8mm
- removed X1: 16MHz, Crystal:Crystal_SMD_SeikoEpson_FA238-4Pin_3.2x2.5mm
- moved J4 38.3 mm to (174.3, 107.4)
Connections:
- J4 pad 1: /D1 -> /D8
- J4 pad 2: /D0 -> /D6
Routing:
- net GND: track 155.5 -> 0.00 mm, vias 13 -> 0
- net VBUS: track 127.1 -> 0.00 mm, vias 8 -> 0
- net /D0: track 120.6 -> 0.00 mm, vias 1 -> 0
- net /D1: track 119.3 -> 0.00 mm, vias 1 -> 0
- net /A0: track 128.5 -> 36.7 mm, vias 2 -> 0
- net /RESET: track 84.0 -> 0.00 mm, vias 3 -> 0
- net /MISO: track 70.7 -> 0.00 mm, vias 5 -> 0
- net /D8: track 95.0 -> 24.6 mm, vias 1 -> 0
- net /D6: track 98.4 -> 30.3 mm, vias 2 -> 0
- net /SCK: track 60.0 -> 0.00 mm, vias 1 -> 0
- net /D7: track 54.1 -> 0.00 mm, vias 2 -> 0
- net /MOSI: track 52.1 -> 0.00 mm, vias 2 -> 0
- net /D3: track 49.6 -> 0.00 mm, vias 1 -> 0
- net /D9: track 44.1 -> 0.00 mm, vias 1 -> 0
- net /D4: track 35.1 -> 0.00 mm, vias 1 -> 0
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- added copper zone on B.Cu, net (none)
- added copper zone on F.Cu, net (none)
- removed copper zone on B.Cu, net GND
- removed copper zone on F.Cu, net GND
Other:
- board size 125.1 x 25.2 mm -> 41.1 x 15 mm
- board text added: "GB3 Extender (100% Gluten Free)"
- board text added: "Pikatea"
- board text removed: "A"
- board text removed: "Pikatea Macropad GB3"
