File: Pikatea Macropad GB3 Addon/Pikatea Macropad GB3 Addon.sch (KiCad schematic (older format))
At the start: 29 parts, among them J1 AVR-ISP-6, J2 USB_B_Mini, J3 Conn_01x03_Male, J4 Conn_01x03_Male, J5 Conn_01x03_Male, J6 Conn_01x06_Male, J7 Conn_01x03_Male, SW1 SW_DPST, SW2 Rotary_Encoder_Switch, U1 ATMEGA32U4-EP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

Commit message: add gb3 addon
Parts:
- removed C1, C10, C2, C3, C4, C5: 0u1, Capacitor_SMD:C_0805_2012Metric, symbol Device:C_Small
- removed C6: 4u7, Capacitor_SMD:C_0805_2012Metric, symbol Device:C_Small
- removed C7, C8: 22p, Capacitor_SMD:C_0805_2012Metric, symbol Device:C_Small
- removed C9: 1u, Capacitor_SMD:C_0805_2012Metric, symbol Device:C_Small
- removed J1: AVR-ISP-6, keyboard_parts:AVR_ICSP_3x2, symbol Connector:AVR-ISP-6
- removed J2: USB_B_Mini, usb_mini:USB-Mini-B_ LCSC-C46398, symbol Connector:USB_B_Mini
- removed J3, J7: Conn_01x03_Male, Connector_PinHeader_2.54mm:PinHeader_1x03_P2.54mm_Vertical, symbol Connector:Conn_01x03_Male
- removed J6: Conn_01x06_Male, Pikatea Macropad Encoder Side Mount:Breakaway-Throughole, symbol Connector:Conn_01x06_Male
- removed MX1, MX2, MX3: MX-LED, MX_Only:MXOnly-1U, symbol MX_Alps_Hybrid:MX-LED
- removed R3: 10K, Resistor_SMD:R_0805_2012Metric, symbol Device:R
- removed R4, R5: 22, Resistor_SMD:R_0805_2012Metric, symbol Device:R
- removed SW1: SW_DPST, Button_Switch_SMD:SW_SPST_TL3342, symbol Switch:SW_DPST
- removed SW2: Rotary_Encoder_Switch, Pikatea Macropad Encoder Side Mount:Encoder-BI_EN11_HSM0E, symbol Device:Rotary_Encoder_Switch
- removed U1: ATMEGA32U4-EP, Package_QFP:LQFP-44_10x10mm_P0.8mm, symbol atmega32u4-ep:ATMEGA32U4-EP
- removed X1: 16MHz, Crystal:Crystal_SMD_SeikoEpson_FA238-4Pin_3.2x2.5mm, symbol Device:Crystal_GND24_Small
Connections:
- net labels removed: CS, D+, D-, D0, D1, D11, D12, D13, D2, D3, D4, GND, MISO, MOSI, RESET, SCK, VBUS, VCC
- wire segments 85 -> 15
- no-connect marks 3 -> 0
