File: FinnGus/FinnGusPCB/FinnGusPCB.kicad_pcb (KiCad board)
At the start: 2 copper layers, 321.4 x 111 mm, 152 parts, among them SW2 Rotary_Encoder_Switch, U2 Teensy2.0_(Arduino)

Commit message: add full kit macropad
Parts:
- MX_57: moved to B.Cu
- turned MX_24 to 280 degrees
- turned MX_57 to 180 degrees
Other:
- board size 321.4 x 111 mm -> 311.4 x 139.6 mm
