File: Pikatea handwire helpers/1u Hand Wire Helpers/1u Hand Wire Helpers.kicad_pcb (KiCad board)
At the start: 2 copper layers, 15.2 x 15.5 mm, 2 parts

Commit message: update handwire helpers
Other:
- net class Default removed
