File: Pikatea R26 macropad/Pikatea R26 Macropad/Pikatea R26 PCB.kicad_pcb (KiCad board)
At the start: 2 copper layers, 118.2 x 46.7 mm, 37 parts, among them J1 AVR-ISP-6, J2 USB_B_Mini, J3 Conn_01x04_Male, J4 Conn_01x04_Male, SW1 SW_DPST, SW2 Rotary_Encoder_Switch, U1 ATMEGA32U4-EP, U2 USBLC6-2P6, Y1 16MHz

Commit message: update R26
Parts:
- MX_1, MX_2, MX_3, MX_4, MX_5, MX_6, MX_7, MX_8: moved to B.Cu
- moved J1 8.95 mm to (119.0, 101.4)
- moved J2 0.40 mm to (99.5, 89.2)
- turned MX_1 to 0 degrees
- turned MX_2 to 0 degrees
- turned MX_3 to 0 degrees
- turned MX_4 to 0 degrees
- turned MX_5 to 0 degrees
- turned MX_6 to 0 degrees
- turned MX_7 to 0 degrees
- turned MX_8 to 0 degrees
Connections:
- J1 pad 1: MISO -> C_5
- U1 pad 10: Net-(U1-Pad10) -> MOSI
- U1 pad 9: Net-(U1-Pad9) -> SCK
Routing:
- net SCK: track 0.00 -> 42.5 mm, vias 0 -> 1
- net MOSI: track 0.00 -> 37.7 mm, vias 0 -> 1
- net VCC: track 104.3 -> 137.9 mm, vias 6 -> 7
- net Reset: track 19.7 -> 48.6 mm, vias 0 -> 2
- net C_5: track 19.7 -> 41.7 mm
- net VCC_USB: track 133.7 -> 116.9 mm
- net C_8: track 20.5 -> 12.5 mm
- net C_6: track 78.3 -> 85.8 mm
- net C_7: track 58.2 -> 65.1 mm
- net GND: track 84.0 -> 90.8 mm, vias 36 -> 45
- net C_9: track 37.0 -> 30.4 mm
- net C_1: track 88.9 -> 95.2 mm
- net C_3: track 28.0 -> 22.4 mm
- net C_2: track 70.6 -> 75.5 mm
- net C_4: track 36.0 -> 31.1 mm
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Other:
- outline, holes or cut-outs redrawn
- board text added: "R26 Proto1"

Commit message: updates
Parts:
- USB1: footprint Type-C:HRO-TYPE-C-31-M-13 -> Type-C:HRO-TYPE-C-31-M-12
Connections:
- U1 pad 8: Net-(U1-Pad8) -> R_1
Routing:
- net R_1: track 191.8 -> 206.7 mm
- net GND: track 90.8 -> 93.7 mm, vias 45 -> 46
- net USB_D-: track 6.41 -> 5.37 mm
- net USB_D+: track 5.64 -> 6.52 mm
- net VCC_USB: track 116.9 -> 116.1 mm
Other:
- board size 118.2 x 46.7 mm -> 118.2 x 45.9 mm
- board text added: "R26 Proto2"
- board text removed: "R26 Proto1"
